File: motor_driver.kicad_pcb (KiCad board)
At the start: 2 copper layers, 30 x 30 mm, 83 parts, among them J1 CAN_IN, J2 CAN_OUT, J3 Battery, J4 Motor, J5 DBG, Q1 SiS415DNT, Q2 SiS454DN, Q3 SiS415DNT, Q4 SiS454DN, Q5 SiS415DNT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

Commit message: finish layout
Parts:
- removed C8: 0u1, Capacitor_SMD:C_0402_1005Metric
- removed C9: 10u, Capacitor_SMD:C_0402_1005Metric
- C10, C16, C17, C19, C21, C24, C28, C29, C31, D10, D5, L1, R1, R2, R20, R21, R22, R4, TP1, U3, U6, U7: moved to B.Cu
- moved R7 134.3 mm to (37.2, 105.5), turned to 180 degrees
- moved R22 131.8 mm to (51.2, 113.8), turned to 180 degrees
- moved R21 131.8 mm to (51.2, 112.8)
- moved D6 130.0 mm to (39.3, 105.5)
- moved R2 91.7 mm to (59.3, 110.5), turned to 180 degrees
- moved C10 91.7 mm to (59.3, 112.5), turned to 180 degrees
- moved R1 88.7 mm to (62.2, 112.5), turned to 180 degrees
- moved D5 78.8 mm to (56.4, 94.5), turned to 90 degrees
- moved D2 78.0 mm to (40.1, 94.3)
- moved R4 72.5 mm to (57.5, 94.5), turned to 90 degrees
- moved C11 70.5 mm to (59.8, 112.0)
- moved U2 70.5 mm to (59.8, 110.2)
- moved D1 70.5 mm to (59.8, 108.4), turned to 180 degrees
- moved R3 67.3 mm to (42.3, 110.6), turned to 90 degrees
- moved TP1 66.9 mm to (55.4, 111.5), turned to 180 degrees
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Connections:
- C25 pad 1: Net-(C25-Pad1) -> Net-(D7-K)
- C26 pad 1: Net-(C26-Pad1) -> Net-(D8-K)
- C27 pad 1: Net-(C27-Pad1) -> Net-(D9-K)
- U5 pad 14: Net-(C27-Pad1) -> Net-(D9-K)
- U5 pad 17: Net-(C26-Pad1) -> Net-(D8-K)
- U5 pad 20: Net-(C25-Pad1) -> Net-(D7-K)
Routing:
- added copper zone on F.Cu, net +BATT
