File: motor_driver.kicad_sch (KiCad schematic)
At the start: 39 parts

Commit message: finish schematic draft, start layout
Parts:
- removed D?: YELLOW, symbol Device:LED
- removed R?: 1K5, symbol Device:R
- added D3: LED, LED_SMD:LED_0402_1005Metric, symbol Device:LED
- added J5: DBG, Connector_JST:JST_GH_SM06B-GHS-TB_1x06-1MP_P1.25mm_Horizontal, symbol Connector_Generic:Conn_01x06
- added R3: 1K5, Resistor_SMD:R_0402_1005Metric, symbol Device:R
- C1, C16, C17, C2, C3, C4, C5, C6, C7, C8, C9: renamed from C?; footprint (none) -> Capacitor_SMD:C_0402_1005Metric
- C10, C15, C18: renamed from C?; footprint Capacitor_SMD:C_0201_0603Metric -> Capacitor_SMD:C_0402_1005Metric
- D2, D4: renamed from D?; footprint (none) -> Diode_SMD:D_SOD-523
- D6: renamed from D?; footprint (none) -> LED_SMD:LED_0402_1005Metric
- J1, J2: renamed from J?; footprint (none) -> Connector_JST:JST_GH_SM04B-GHS-TB_1x04-1MP_P1.25mm_Horizontal
- R2: renamed from R?; footprint Resistor_SMD:R_0201_0603Metric -> Resistor_SMD:R_0402_1005Metric
- R7: renamed from R?; footprint (none) -> Resistor_SMD:R_0402_1005Metric
- TP1: renamed from TP?; footprint (none) -> TestPoint:TestPoint_Pad_1.0x1.0mm
- U3: renamed from U?; footprint Package_DFN_QFN:QFN-16-1EP_3x3mm_P0.5mm_EP1.8x1.8mm -> Package_DFN_QFN:QFN-16-1EP_3x3mm_P0.5mm_EP1.7x1.7mm
- Y1: renamed from Y?; value 12MHz -> 16MHz
- gave numbers to parts that had none: 13
Connections:
- net CAN1_SILENT is gone; now on net CAN_SILENT: U1.45 (PB7)
- net CAN_H is gone; now on net CAN_P: J1.2 (Pin_2), J2.2 (Pin_2)
- net CAN_L is gone; now on net CAN_N: J1.3 (Pin_3), J2.3 (Pin_3)
- net +3V3: now also J5.1 (Pin_1)
- net GND: now also J5.6 (Pin_6), R3.2
- net STATUS: now also D3.2 (A)
- net SWCLK: now also J5.5 (Pin_5)
- net SWDIO: now also J5.4 (Pin_4)
- net USART3_RX_DBG: now also J5.3 (Pin_3)
- net USART3_TX_DBG: now also J5.2 (Pin_2)
- new net: D3.1 (K), R3.1
Other:
- sheet Power Stage ports: added 3V3_SENSE, VIN1M, VIN1P, VIN2M, VIN2P, VIN3M, VIN3P; removed OPAMP1_VINM, OPAMP1_VINP, OPAMP2_VINM, OPAMP2_VINP, OPAMP3_VINM, OPAMP3_VINP
- note added: "CAN & Debug Connectors"
- note added: "Power Stage"
- note removed: "CAN Connectors"
- moved on the sheet: C16, C17, D2, D4, J1, J2, U3

Commit message: finish layout
Parts:
- removed C8: 0u1, Capacitor_SMD:C_0402_1005Metric, symbol Device:C
- removed C9: 10u, Capacitor_SMD:C_0402_1005Metric, symbol Device:C
Connections:
- no-connect marks 18 -> 22
Other:
- moved on the sheet: C7
